File: boards/Main PCB/Main.sch (EAGLE design)
At the start: 90 parts, among them CN1 MINIB, CN2 MINIB, IC1 FT232RL, IC2 FT232RL, J1 3_PIN_JST-XH, J2 2_PIN_JST-XH, Q4 BSS138, Q5 BSS138, Q6 BSS138, Q7 BSS138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

Commit message: Fixing IMU traces and adding descriptive net names
Parts:
- removed JP2: (no value), microbuilder:HEADER-1X476MIL
Connections:
- net N$12 renamed D+_LIDAR
- net N$13 renamed D-_LIDAR
- net N$20 renamed ENCODER1
- net N$21 renamed ENCODER2
- net N$25 renamed US1_ECHO
- net N$3 renamed D+_GPS
- net N$38 renamed 12V_IN
- net N$4 renamed D-_GPS
- net N$44 renamed US3_TRIG
- net N$45 renamed US3_ECHO
- net N$46 renamed US2_TRIG
- net N$50 renamed US1_TRIG
- net N$54 renamed US2_ECHO
- net I2CADDR_3V: no longer JP2.4
- net INT_3V: no longer JP2.3
- net PS0_3V: no longer JP2.1
- net PS1_3V: no longer JP2.2
Changed lines of the file:
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@@
 <?xml version="1.0" encoding="utf-8"?>
 <!DOCTYPE eagle SYSTEM "eagle.dtd">
-<eagle version="9.3.0">
+<eagle version="9.2.2">
 <drawing>
 <settings>
@@
 <part name="U$21" library="microbuilder" deviceset="3.3V" device=""/>
 <part name="U$15" library="microbuilder" deviceset="3.3V" device=""/>
-<part name="JP2" library="microbuilder" deviceset="HEADER-1X4" device="76MIL"/>
 <part name="U$1" library="NS-HP-GL" deviceset="GPS" device=""/>
 <part name="CN2" library="adafruit" deviceset="USB" device="MINIB" value="MINIB"/>
@@
 </segment>
 </net>
-<net name="N$3" class="0">
+<net name="D+_GPS" class="0">
 <segment>
 <wire x1="38.1" y1="93.98" x2="45.72" y2="93.98" width="0.1524" layer="91"/>
@@
 <pinref part="CN1" gate="G$1" pin="D+"/>
 <pinref part="IC1" gate="1" pin="USBDP"/>
-</segment>
-</net>
-<net name="N$4" class="0">
+<label x="38.1" y="93.98" size="1.778" layer="95"/>
+</segment>
+</net>
+<net name="D-_GPS" class="0">
 <segment>
 <wire x1="83.82" y1="60.96" x2="43.18" y2="60.96" width="0.1524" layer="91"/>
@@
 <pinref part="IC1" gate="1" pin="USBDM"/>
 <pinref part="CN1" gate="G$1" pin="D-"/>
+<label x="38.1" y="91.44" size="1.778" layer="95"/>
 </segment>
 </net>
@@
 </segment>
 </net>
-<net name="N$12" class="0">
+<net name="D+_LIDAR" class="0">
 <segment>
 <wire x1="43.18" y1="86.36" x2="50.8" y2="86.36" width="0.1524" layer="91"/>
@@
 <pinref part="CN2" gate="G$1" pin="D+"/>
 <pinref part="IC2" gate="1" pin="USBDP"/>
-</segment>
-</net>
-<net name="N$13" class="0">
+<label x="43.18" y="86.36" size="1.778" layer="95"/>
+</segment>
+</net>
+<net name="D-_LIDAR" class="0">
 <segment>
 <wire x1="88.9" y1="53.34" x2="48.26" y2="53.34" width="0.1524" layer="91"/>
@@
 <pinref part="IC2" gate="1" pin="USBDM"/>
 <pinref part="CN2" gate="G$1" pin="D-"/>
+<label x="43.18" y="83.82" size="1.778" layer="95"/>
 </segment>
 </net>
@@
 </busses>
 <nets>
-<net name="N$25" class="0">
+<net name="US1_ECHO" class="0">
 <segment>
 <pinref part="U2" gate="G$1" pin="PA1/USART2_RTS/TIM15_CH1N/USART4_RX/EVENTOUT/ADC_IN1"/>
@@
 <wire x1="40.894" y1="196.088" x2="40.894" y2="198.628" width="0.1524" layer="91"/>
 <junction x="40.894" y="198.628"/>
-</segment>
-</net>
-<net name="N$21" class="0">
+<label x="160.02" y="144.78" size="1.778" layer="95"/>
+</segment>
+</net>
+<net name="ENCODER2" class="0">
 <segment>
 <pinref part="U2" gate="G$1" pin="PB1/TIM3_CH4/USART3_RTS/TIM14_CH1/TIM1_CH3N/ADC_IN9"/>
@@
 <pinref part="X7" gate="-2" pin="S"/>
 <wire x1="386.08" y1="139.7" x2="408.94" y2="139.7" width="0.1524" layer="91"/>
+<label x="350.52" y="144.78" size="1.778" layer="95"/>
 </segment>
 </net>
@@
 </segment>
 </net>
-<net name="N$20" class="0">
+<net name="ENCODER1" class="0">
 <segment>
 <pinref part="U2" gate="G$1" pin="PB0/TIM3_CH3/TIM1_CH2N/EVENTOUT/USART3_CK/ADC_IN8"/>
@@
 <pinref part="X6" gate="-2" pin="S"/>
 <wire x1="401.32" y1="160.02" x2="408.94" y2="160.02" width="0.1524" layer="91"/>
+<label x="350.52" y="147.32" size="1.778" layer="95"/>
 </segment>
 </net>
@@
 </segment>
 </net>
-<net name="N$38" class="0">
+<net name="12V_IN" class="0">
 <segment>
 <pinref part="J2" gate="G$1" pin="P$2"/>
@@
 <wire x1="0" y1="259.08" x2="5.08" y2="259.08" width="0.1524" layer="91"/>
 <junction x="0" y="259.08"/>
+<label x="-10.16" y="259.08" size="1.778" layer="95"/>
 </segment>
 </net>
@@
 </segment>
 </net>
-<net name="N$44" class="0">
+<net name="US3_TRIG" class="0">
 <segment>
 <wire x1="96.52" y1="109.22" x2="96.52" y2="132.08" width="0.1524" layer="91"/>
@@
 <wire x1="96.52" y1="109.22" x2="35.56" y2="109.22" width="0.1524" layer="91"/>
 <junction x="35.56" y="109.22"/>
+<label x="160.02" y="132.08" size="1.778" layer="95"/>
 </segment>
 </net>
@@
 </segment>
 </net>
-<net name="N$46" class="0">
+<net name="US2_TRIG" class="0">
 <segment>
 <wire x1="114.3" y1="144.78" x2="114.3" y2="137.16" width="0.1524" layer="91"/>
@@
 <wire x1="35.56" y1="144.78" x2="35.56" y2="154.94" width="0.1524" layer="91"/>
 <junction x="35.56" y="154.94"/>
+<label x="160.02" y="137.16" size="1.778" layer="95"/>
 </segment>
 </net>
@@
 </segment>
 </net>
-<net name="N$50" class="0">
+<net name="US1_TRIG" class="0">
 <segment>
 <wire x1="119.38" y1="182.88" x2="119.38" y2="147.32" width="0.1524" layer="91"/>
@@
 <wire x1="35.56" y1="182.88" x2="35.56" y2="203.2" width="0.1524" layer="91"/>
 <junction x="35.56" y="203.2"/>
+<label x="160.02" y="147.32" size="1.778" layer="95"/>
 </segment>
 </net>
@@
 </segment>
 </net>
-<net name="N$54" class="0">
+<net name="US2_ECHO" class="0">
 <segment>
 <pinref part="Q5" gate="G$1" pin="S"/>
@@
 <wire x1="111.76" y1="150.368" x2="111.76" y2="134.62" width="0.1524" layer="91"/>
 <junction x="40.894" y="150.368"/>
-</segment>
-</net>
-<net name="N$45" class="0">
+<label x="160.02" y="134.62" size="1.778" layer="95"/>
+</segment>
+</net>
+<net name="US3_ECHO" class="0">
 <segment>
 <pinref part="R27" gate="G$1" pin="1"/>
@@
 <wire x1="99.06" y1="104.648" x2="99.06" y2="129.54" width="0.1524" layer="91"/>
 <junction x="40.894" y="104.648"/>
+<label x="160.02" y="129.54" size="1.778" layer="95"/>
 </segment>
 </net>
@@
 <instance part="U$15" gate="G$1" x="-25.4" y="-25.4" smashed="yes" rot="R270">
 <attribute name="VALUE" x="-24.384" y="-23.876" size="1.27" layer="96" rot="R270"/>
-</instance>
-<instance part="JP2" gate="A" x="55.88" y="-40.64" smashed="yes">
-<attribute name="NAME" x="49.53" y="-32.385" size="1.778" layer="95"/>
-<attribute name="VALUE" x="49.53" y="-48.26" size="1.778" layer="96"/>
 </instance>
 <instance part="FRAME1" gate="G$1" x="-127" y="-124.46" smashed="yes"/>
@@
 </segment>
 <segment>
-<wire x1="33.02" y1="-38.1" x2="53.34" y2="-38.1" width="0.1524" layer="91"/>
-<label x="33.02" y="-38.1" size="1.778" layer="95"/>
-<pinref part="JP2" gate="A" pin="2"/>
-</segment>
-<segment>
 <pinref part="JP4" gate="A" pin="3"/>
 <wire x1="-5.08" y1="-58.42" x2="20.32" y2="-58.42" width="0.1524" layer="91"/>
@@
 </segment>
 <segment>
-<wire x1="33.02" y1="-35.56" x2="53.34" y2="-35.56" width="0.1524" layer="91"/>
-<label x="33.02" y="-35.56" size="1.778" layer="95"/>
-<pinref part="JP2" gate="A" pin="1"/>
-</segment>
-<segment>
 <pinref part="JP4" gate="A" pin="4"/>
 <wire x1="-5.08" y1="-55.88" x2="20.32" y2="-55.88" width="0.1524" layer="91"/>
@@
 <wire x1="-30.48" y1="-7.62" x2="-17.78" y2="-7.62" width="0.1524" layer="91"/>
 <label x="-27.94" y="-7.62" size="1.778" layer="95"/>
-</segment>
-<segment>
-<wire x1="33.02" y1="-40.64" x2="53.34" y2="-40.64" width="0.1524" layer="91"/>
-<label x="33.02" y="-40.64" size="1.778" layer="95"/>
-<pinref part="JP2" gate="A" pin="3"/>
 </segment>
 <segment>
@@
 </segment>
 <segment>
-<wire x1="33.02" y1="-43.18" x2="53.34" y2="-43.18" width="0.1524" layer="91"/>
-<label x="33.02" y="-43.18" size="1.778" layer="95"/>
-<pinref part="JP2" gate="A" pin="4"/>
-</segment>
-<segment>

Commit message: More routing and naming improvements
Connections:
- net N$40 renamed SABERTOOTH_S1
- net N$41 renamed SABERTOOTH_5V
- net N$42 renamed SABERTOOTH_GND
Changed lines of the file:
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@@
 <?xml version="1.0" encoding="utf-8"?>
 <!DOCTYPE eagle SYSTEM "eagle.dtd">
-<eagle version="9.2.2">
+<eagle version="9.3.0">
 <drawing>
 <settings>
@@
 </segment>
 </net>
-<net name="N$40" class="0">
+<net name="SABERTOOTH_S1" class="0">
 <segment>
 <pinref part="J1" gate="G$1" pin="P$1"/>
@@
 </segment>
 </net>
-<net name="N$41" class="0">
+<net name="SABERTOOTH_5V" class="0">
 <segment>
 <pinref part="R20" gate="G$1" pin="1"/>
@@
 </segment>
 </net>
-<net name="N$42" class="0">
+<net name="SABERTOOTH_GND" class="0">
 <segment>
 <pinref part="J1" gate="G$1" pin="P$3"/>

Commit message: Minor routing improvements and net naming
Connections:
- net SABERTOOTH_5V: now also J1.P$1, R20.2; no longer J1.P$2, R20.1, U3.C_T
- net SABERTOOTH_S1: now also J1.P$2, R20.1, U3.C_T; no longer J1.P$1, R20.2
Changed lines of the file:
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@@
 <?xml version="1.0" encoding="utf-8"?>
 <!DOCTYPE eagle SYSTEM "eagle.dtd">
-<eagle version="9.3.0">
+<eagle version="9.2.2">
 <drawing>
 <settings>
@@
 </segment>
 </net>
-<net name="SABERTOOTH_S1" class="0">
+<net name="SABERTOOTH_5V" class="0">
 <segment>
 <pinref part="J1" gate="G$1" pin="P$1"/>
@@
 </segment>
 </net>
-<net name="SABERTOOTH_5V" class="0">
+<net name="SABERTOOTH_S1" class="0">
 <segment>
 <pinref part="R20" gate="G$1" pin="1"/>
